File: breakout-ttgf0p1-adapter.kicad_pcb (KiCad board)
At the start: 4 copper layers, 50 x 50 mm, 118 parts, among them J1 Conn_01x12, J2 Conn_02x08_Odd_Even, J3 DF12NB-60DS-0.5V_51, J4 Conn_02x08_Odd_Even, J5 DF12NB-50DS-0.5V_51, J6 Conn_02x08_Odd_Even, J8 Conn_02x08_Odd_Even, U1 AP2112K-3.3, U2 AP2112K-3.3, U4 24LC02

Commit message: update component fields
Parts:
- C10, C11, C12, C13, C14, C15, C16, C17: value 1u -> 1uF
- R10, R11: value 1k -> 1kΩ
- R2, R3, R4, R6, R7, R8: value 0 -> 0Ω
Changed lines of the file:
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@@
 			)
 		)
-		(property "Datasheet" ""
+		(property "Datasheet" "~"
 			(at 0 0 90)
 			(layer "F.Fab")
@@
 			)
 		)
-		(property "Description" ""
+		(property "Description" "Generic connector, double row, 02x08, odd/even pin numbering scheme (row 1 odd numbers, row 2 even numbers), script generated (kicad-library-utils/schlib/autogen/connector/)"
 			(at 0 0 90)
 			(layer "F.Fab")
@@
 			)
 		)
+		(property ki_fp_filters "Connector*:*_2x??_*")
+		(sheetname "/")
+		(sheetfile "breakout-ttgf0p1-adapter.kicad_sch")
 		(attr smd)
 		(fp_line
@@
 			)
 		)
-		(property "Datasheet" ""
+		(property "Datasheet" "~"
 			(at 0 0 0)
 			(layer "F.Fab")
@@
 			)
 		)
-		(property "Description" ""
+		(property "Description" "Generic connector, double row, 02x08, odd/even pin numbering scheme (row 1 odd numbers, row 2 even numbers), script generated (kicad-library-utils/schlib/autogen/connector/)"
 			(at 0 0 0)
 			(layer "F.Fab")
@@
 			)
 		)
+		(property ki_fp_filters "Connector*:*_2x??_*")
+		(sheetname "/")
+		(sheetfile "breakout-ttgf0p1-adapter.kicad_sch")
 		(attr smd)
 		(fp_line
@@
 			)
 		)
-		(property "Value" "0"
+		(property "Value" "0Ω"
 			(at 0 1.65 0)
 			(layer "F.Fab")
@@
 			)
 		)
-		(property "LCSC" "C4143065"
+		(property "LCSC" "C17477"
 			(at 0 0 180)
 			(unlocked yes)
@@
 			)
 		)
-		(property "Value" "1u"
+		(property "Value" "1uF"
 			(at 0 1.16 0)
 			(layer "F.Fab")
@@
 			)
 		)
-		(property "Value" "1u"
+		(property "Value" "1uF"
 			(at 0 1.16 0)
 			(layer "F.Fab")
@@
 			)
 		)
-		(property "Value" "1u"
+		(property "Value" "1uF"
 			(at 0 1.16 90)
 			(layer "F.Fab")
@@
 			)
 		)
-		(property "Value" "0"
+		(property "Value" "0Ω"
 			(at 0 1.43 90)
 			(layer "F.Fab")
@@
 			)
 		)
-		(property "LCSC" "C95177"
+		(property "LCSC" " C21189"
 			(at 0 0 270)
 			(unlocked yes)
@@
 			)
 		)
-		(property "Value" "1k"
+		(property "Value" "1kΩ"
 			(at 0 1.17 90)
 			(layer "F.Fab")
@@
 			)
 		)
-		(property "Value" "1u"
+		(property "Value" "1uF"
 			(at 0 1.16 90)
 			(layer "F.Fab")
@@
 			)
 		)
-		(property "Value" "0"
+		(property "Value" "0Ω"
 			(at 0 1.65 0)
 			(layer "F.Fab")
@@
 			)
 		)
-		(property "LCSC" "C4143065"
+		(property "LCSC" "C17477"
 			(at 0 0 180)
 			(unlocked yes)
@@
 			)
 		)
-		(property "Datasheet" ""
+		(property "Datasheet" "~"
 			(at 0 0 90)
 			(layer "F.Fab")
@@
 			)
 		)
-		(property "Description" ""
+		(property "Description" "Generic connector, double row, 02x08, odd/even pin numbering scheme (row 1 odd numbers, row 2 even numbers), script generated (kicad-library-utils/schlib/autogen/connector/)"
 			(at 0 0 90)
 			(layer "F.Fab")
@@
 			)
 		)
+		(property ki_fp_filters "Connector*:*_2x??_*")
+		(sheetname "/")
+		(sheetfile "breakout-ttgf0p1-adapter.kicad_sch")
 		(attr smd)
 		(fp_line
@@
 			)
 		)
-		(property "Value" "1u"
+		(property "Value" "1uF"
 			(at 0 1.16 0)
 			(layer "F.Fab")
@@
 			)
 		)
-		(property "Value" "0"
+		(property "Value" "0Ω"
 			(at 0 1.43 90)
 			(layer "F.Fab")
@@
 			)
 		)
-		(property "LCSC" ""
+		(property "LCSC" " C21189"
 			(at 0 0 270)
 			(unlocked yes)
@@
 			)
 		)
-		(property "Value" "1u"
+		(property "Value" "1uF"
 			(at 0 1.16 90)
 			(layer "F.Fab")
@@
 			)
 		)
-		(property "Value" "1k"
+		(property "Value" "1kΩ"
 			(at 0 1.17 90)
 			(layer "F.Fab")
@@
 			)
 		)
-		(property "Value" "1u"
+		(property "Value" "1uF"
 			(at 0 1.16 0)
 			(layer "F.Fab")
@@
 			)
 		)
-		(property "Value" "0"
+		(property "Value" "0Ω"
 			(at 0 1.43 0)
 			(layer "F.Fab")
@@
 			)
 		)
-		(property "LCSC" "C95177"
+		(property "LCSC" " C21189"
 			(at 0 0 180)
 			(unlocked yes)
@@
 			)
 		)
-		(property "Value" "0"
+		(property "Value" "0Ω"
 			(at 0 1.43 0)
 			(layer "F.Fab")
@@
 			)
 		)
-		(property "LCSC" "C95177"
+		(property "LCSC" " C21189"
 			(at 0 0 180)
 			(unlocked yes)
@@
 			)
 		)
-		(property "Datasheet" ""
+		(property "Datasheet" "~"
 			(at 0 0 0)
 			(layer "F.Fab")
@@
 			)
 		)
-		(property "Description" ""
+		(property "Description" "Generic connector, double row, 02x08, odd/even pin numbering scheme (row 1 odd numbers, row 2 even numbers), script generated (kicad-library-utils/schlib/autogen/connector/)"
 			(at 0 0 0)
 			(layer "F.Fab")
@@
 			)
 		)
+		(property ki_fp_filters "Connector*:*_2x??_*")
+		(sheetname "/")
+		(sheetfile "breakout-ttgf0p1-adapter.kicad_sch")
 		(attr smd)
 		(fp_line
@@
 			)
 		)
-		(property "Value" "1u"
+		(property "Value" "1uF"
 			(at 0 1.16 90)
 			(layer "F.Fab")
